File: KiCAD/fyp_nubots_ssl/analogue.kicad_sch (KiCad schematic)
At the start: 29 parts, among them U2 AD7606

Commit message: Submitted final report.
Parts:
- removed C16: 100n, Capacitor_SMD:C_0603_1608Metric, symbol Device:C
- removed R14, R16, R17, R18, R19, R20, R22, R23, R24, R25: 10k, Resistor_SMD:R_0603_1608Metric, symbol Device:R_US
- added C23, C31: 100n, Capacitor_SMD:C_0603_1608Metric, symbol Device:C
- added C5: 4.7p, Capacitor_SMD:C_0603_1608Metric, symbol Device:C
- added R13: 10k, Resistor_SMD:R_0603_1608Metric, symbol Device:R_US
- added U5: TLV272, Package_SO:MSOP-8_3x3mm_P0.65mm, symbol Device:Opamp_Dual
- C21: renamed from C17; footprint Capacitor_SMD:C_0603_1608Metric -> Capacitor_SMD:C_0805_2012Metric
- C25: renamed from C19; footprint Capacitor_SMD:C_0603_1608Metric -> Capacitor_SMD:C_0805_2012Metric
- C26: renamed from C21; footprint Capacitor_SMD:C_0603_1608Metric -> Capacitor_SMD:C_0805_2012Metric
- C27: renamed from C22; footprint Capacitor_SMD:C_0603_1608Metric -> Capacitor_SMD:C_0805_2012Metric
- C28: renamed from C20; footprint Capacitor_SMD:C_0603_1608Metric -> Capacitor_SMD:C_0805_2012Metric
- renumbered C13 to C18, C15 to C19, C18 to C20, C14 to C22, R13 to R14, R11 to R16, R10 to R17, R9 to R18, R8 to R19, R12 to R20
Connections:
- net +3V3: now also R21.2; no longer R17.1, R18.1, R19.1
- net +5V: now also C23.1, C31.1, U5.8 (V+)
- net CONVST: now also C5.1, R13.2; no longer U2.10 (CONVST_B)
- net GNDA: now also R17.2, R18.2, R19.2, C23.2, C31.2, U5.4 (V-); no longer R21.1
- net at U2.3 (OS0): now also R17.1; no longer R19.2
- net DB13: now reaches U2.31 (DB13)
- net DB1: now reaches U2.17 (DB1)
- net DB5: now reaches U2.21 (DB5)
- net DB0: now reaches U2.16 (DB0)
- net at R15.2: now also U2.6 (~{PAR}/SER/BYTE_SEL); no longer U2.30 (DB12)
- net DB2: now reaches U2.18 (DB2)
- net DB2: no longer R21.2
- net DB3: now reaches U2.19 (DB3)
- net DB4: now reaches U2.20 (DB4)
- net DB6: now reaches U2.22 (DB6)
- net DB14: now reaches U2.32 (DB14/HBEN)
- net DB15: now reaches U2.33 (DB15/BYTE_SEL)
- net at U2.4 (OS1): now also R18.1; no longer R18.2
- net REFOUT: now reaches C25.1, U2.42 (REFIN/REFOUT)
- net REFOUT: now also U5.3 (+)
- net channels_12/CH1+: now reaches U2.49 (V1)
- net at U2.5 (OS2): now also R19.1; no longer R17.2
- net channels_12/CH1-: now reaches U2.50 (V1GND)
- net channels_12/CH2+: now reaches U2.51 (V2)
- net channels_12/CH2-: now reaches U2.52 (V2GND)
- net channels_34/CH1+: now reaches U2.53 (V3)
- net channels_34/CH1-: now reaches U2.54 (V3GND)
- net channels_34/CH2+: now reaches U2.55 (V4)
- net channels_34/CH2-: now reaches U2.56 (V4GND)
- net channels_56/CH1+: now reaches U2.57 (V5)
- net channels_56/CH1-: now reaches U2.58 (V5GND)
- net channels_56/CH2+: now reaches U2.59 (V6)
- net channels_56/CH2-: now reaches U2.60 (V6GND)
- net channels_78/CH1+: now reaches U2.61 (V7)
- net channels_78/CH1-: now reaches U2.62 (V7GND)
- net channels_78/CH2+: now reaches U2.63 (V8)
- net channels_78/CH2-: now reaches U2.64 (V8GND)
- net DOUT_A renamed DB7
- net DOUT_B renamed DB8
- net DOUT_C renamed DB10
- net DB10: no longer U2.27 (DB9)
- net SDI renamed DB11
- net /CS renamed nCS
- new net DB12: U2.30 (DB12)
- new net DB9: U2.27 (DB9)
- new net GND: C5.2, R13.1
- new net REF: U5.1, U5.2 (-)
- new net nWR: R21.1, U2.10 (CONVST_B)
- no-connect marks 0 -> 3
Other:
- added sheet channels_12 (channels.kicad_sch)
- added sheet channels_34 (channels.kicad_sch)
- added sheet channels_56 (channels.kicad_sch)
- added sheet channels_78 (channels.kicad_sch)
- moved on the sheet: C18, C19, C20, C21, C22, C25, C26, C27, C28, R14, R16, R17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
