File: KiCAD/fyp_nubots_ssl/fyp_nubots_ssl.kicad_sch (KiCad schematic)
At the start: 0 parts

Commit message: Submitted final report.
Parts:
- added C1, C3: 0.33μF, Capacitor_SMD:C_1206_3216Metric, symbol Device:C
- added C2, C4: 0.1μF, Capacitor_SMD:C_1206_3216Metric, symbol Device:C
- added C59, C60: 1μ, Capacitor_SMD:C_0603_1608Metric, symbol Device:C
- added C61: 10n, Capacitor_SMD:C_0603_1608Metric, symbol Device:C
- added D1 (x2): LED, LED_SMD:LED_0805_2012Metric, symbol Device:LED
- added J1: Conn_01x04_Pin, Connector_Molex:Molex_SPOX_5267-04A_1x04_P2.50mm_Vertical, symbol Connector:Conn_01x04_Pin
- added J2: Screw_Terminal_01x02, TerminalBlock:TerminalBlock_bornier-2_P5.08mm, symbol Connector:Screw_Terminal_01x02
- added R1: 1.5k, Resistor_SMD:R_0603_1608Metric, symbol Device:R_US
- added R2: 650, Resistor_SMD:R_0603_1608Metric, symbol Device:R_US
- added R72, R73, R74, R75: 0, Resistor_SMD:R_1206_3216Metric, symbol Device:R_US
- added U1: L78M05, Package_TO_SOT_SMD:TO-252-2, symbol Regulator_Linear:L78M05
- added U2: UA78M33, Package_TO_SOT_SMD:TO-252-2, symbol Regulator_Linear:UA78M33
- added U9: LD3985M18R_SOT23, Package_TO_SOT_SMD:SOT-23-5_HandSoldering, symbol Regulator_Linear:LD3985M18R_SOT23
Connections:
- new net: C59.2, R74.1, U9.5 (VOUT)
- new net: C3.2, R72.2, R73.2, U2.1 (IN)
- new net: C61.2, U9.4 (BYP)
- new net: C2.2, R75.1, U1.3 (OUT)
- new net: D1.2 (A), R2.1
- new net: D1.2 (A), R1.1
- new net +3V3: C4.2, R2.2, U2.3 (OUT)
- new net +5V: R1.2, R73.1, R74.2, R75.2
- new net +5VD: C60.2, R72.1, U9.1 (VIN), U9.3 (INH)
- new net GND: C1.1, C2.1, C3.1, C4.1, C59.1, C60.1, C61.1, D1.1 (K), D1.1 (K), J1.4 (Pin_4), J2.1 (Pin_1), U1.2 (GND), U2.2 (GND), U9.2 (GND)
- new net V_IN: C1.2, J1.3 (Pin_3), J2.2 (Pin_2), U1.1 (IN)
- no-connect marks 0 -> 2
Other:
- sheet analogue ports: added DB[0..15], nCS, nWR; removed DOUT_A, DOUT_B, DOUT_C, SDI, /CS
- sheet processor ports: added BUSY, CONVST, DB[0..15], FRSTDATA, RESET, SCLK, nCS, nWR; removed none
