File: KiCAD/fyp_nubots_ssl/processor.kicad_sch (KiCad schematic)
At the start: 25 parts, among them J1 Conn_02x05_Odd_Even, SW1 SW_Omron_B3FS, SW2 SW_Omron_B3FS, U1 STM32H723VGTx, U3 THVD1400D

Commit message: Submitted final report.
Parts:
- removed C1 (x2), C5: 100n, Capacitor_SMD:C_0603_1608Metric, symbol Device:C
- removed R1: 10k, Resistor_SMD:R_0603_1608Metric, symbol Device:R_US
- removed R2: 47, Resistor_SMD:R_0603_1608Metric, symbol Device:R_US
- removed U3: THVD1400D, Package_SO:SOIC-14_3.9x8.7mm_P1.27mm, symbol Interface_UART:THVD1400D
- added C1, C5: 100n, Capacitor_SMD:C_0603_1608Metric, symbol Device:C
- added C29, C30: 5.6p, Capacitor_SMD:C_0402_1005Metric, symbol Device:C
- added C5: 4.7n, Capacitor_SMD:C_0603_1608Metric, symbol Device:C
- added D3: LED, LED_SMD:LED_0805_2012Metric, symbol Device:LED
- added J3: USB_B_Micro, Connector_USB:USB_Micro-B_Amphenol_10118193-0001LF_Horizontal, symbol Connector:USB_B_Micro
- added J5: Conn_02x06_Odd_Even, Connector_PinHeader_2.54mm:PinHeader_2x06_P2.54mm_Vertical, symbol Connector_Generic:Conn_02x06_Odd_Even
- added R1: 1.5k, Resistor_SMD:R_0603_1608Metric, symbol Device:R_US
- added R1: 1M, Resistor_SMD:R_0603_1608Metric, symbol Device:R_US
- added R1, R2: 10k, Resistor_SMD:R_0603_1608Metric, symbol Device:R_US
- added R2: 650, Resistor_SMD:R_0603_1608Metric, symbol Device:R_US
- added R22, R23: 0, Resistor_SMD:R_0402_1005Metric, symbol Device:R_US
- added Y1: Crystal_GND24, Crystal:Crystal_SMD_2520-4Pin_2.5x2.0mm, symbol Device:Crystal_GND24
- C12: value 100n -> 4.7μ; footprint Capacitor_SMD:C_0603_1608Metric -> Capacitor_SMD:C_0805_2012Metric
- C6: value 4.7μ -> 100n; footprint Capacitor_SMD:C_1206_3216Metric -> Capacitor_SMD:C_0603_1608Metric
- C7: value 100n -> 1μ; footprint Capacitor_SMD:C_0603_1608Metric -> Capacitor_SMD:C_0805_2012Metric
- C8: value 1μ -> 100n; footprint Capacitor_SMD:C_1206_3216Metric -> Capacitor_SMD:C_0603_1608Metric
- R3: value 10k -> 47; footprint (none) -> Resistor_SMD:R_0603_1608Metric
- R4, R5, R6: footprint (none) -> Resistor_SMD:R_0603_1608Metric
Connections:
- net +3V3: now also C10.1, C11.1, C12.1, R3.2, R6.1, C5.1, R1.1, R1.1, R2.1; no longer C2.1, C3.1, R3.1, R5.1
- net BOOT: now also SW2.2, R2.2; no longer SW1.2
- net GND: now also C11.2, C2.1, R5.2, C1.2, C29.2, C30.2, C5.2, C5.2, D3.1 (K), J3.4 (ID), J3.5 (GND), J5.1 (Pin_1), J5.11 (Pin_11), J5.3 (Pin_3), J5.5 (Pin_5), J5.7 (Pin_7), J5.9 (Pin_9), R1.2, Y1.2, Y1.4; no longer C11.1, C2.2, R6.2
- net JTCK_SWCLK: now also R5.1; no longer R6.1
- net JTDI: now also R7.2; no longer R5.2, U1.77 (PA15(JTDI))
- net JTDO_SWO: now also R6.2; no longer R4.2, U1.89 (PB3(JTDO)
- net JTMS_SWDIO: now also R4.2; no longer R3.2
- net NJTRST: no longer U1.90 (PB4(NJTRST))
- net NRST: now also SW1.2, C1.1, R1.2; no longer C10.1, R7.2, SW2.2
- net at U1.20 (VREF+): now also R3.1
- net at U1.48 (VCAP): now also C2.2; no longer C11.2
- net at U1.73 (VCAP): now also C3.1; no longer C12.1
- net PH0_OSC_IN: now reaches U1.12 (PH0)
- net PH0_OSC_IN: now also R22.2
- net PH1_OSC_OUT: now reaches U1.13 (PH1)
- net PH1_OSC_OUT: now also R23.2
- net CONVST: now reaches U1.22 (PA0)
- net CONVST: now also J5.2 (Pin_2)
- net nCS: now reaches U1.30 (PA6)
- net nCS: now also J5.6 (Pin_6)
- net DB8: now reaches U1.55 (PD8)
- net DB9: now reaches U1.56 (PD9)
- net DB10: now reaches U1.57 (PD10)
- net DB11: now reaches U1.58 (PD11)
- net DB12: now reaches U1.59 (PD12)
- net DB13: now reaches U1.60 (PD13)
- net DB14: now reaches U1.61 (PD14)
- net DB15: now reaches U1.62 (PD15)
- net DB15: now also J5.12 (Pin_12)
- net SCLK: now reaches U1.63 (PC6)
- net SCLK: now also J5.4 (Pin_4)
- net BUSY: now reaches U1.64 (PC7)
- net BUSY: now also J5.8 (Pin_8)
- net FRSTDATA: now reaches U1.65 (PC8)
- net FRSTDATA: now also J5.10 (Pin_10)
- net RESET: now reaches U1.66 (PC9)
- net nWR: now reaches U1.67 (PA8)
- net USB_OTG_HS_DM: now reaches U1.70 (PA11)
- net USB_OTG_HS_DM: now also J3.2 (D-)
- net USB_OTG_HS_DP: now reaches U1.71 (PA12)
- net USB_OTG_HS_DP: now also J3.3 (D+), R1.2
- net LED_0: now reaches U1.78 (PC10)
- net LED_0: now also R2.2
- net DB0: now reaches U1.81 (PD0)
- net DB1: now reaches U1.82 (PD1)
- net DB2: now reaches U1.83 (PD2)
- net DB3: now reaches U1.84 (PD3)
- net DB4: now reaches U1.85 (PD4)
- net DB5: now reaches U1.86 (PD5)
- net DB6: now reaches U1.87 (PD6)
- net DB7: now reaches U1.88 (PD7)
- new net: C5.1, J3.6 (Shield), R1.1
- new net: D3.2 (A), R2.1
- new net: C30.1, R23.1, Y1.3
- new net: C29.1, R22.1, Y1.1
- new net +5VD: J3.1 (VBUS)
- no-connect marks 0 -> 52
